File: Hardware/STM32.sch (KiCad schematic (older format))
At the start: 0 parts

Commit message: Base ESP32 sheet done. STM32 in place
Parts:
- added C? (x3): 4.7uF, symbol C
- added C? (x5): 100nF, symbol C
- added C?: 1uF, symbol C
- added C?: 10nF, symbol C
- added U?: STM32F042C6T6, QFP50P700X700X160-48N, symbol STM32F042C6T6
Connections:
- new net +3V3: C?.1, C?.1, C?.1, C?.1, C?.1, C?.1, C?.1, C?.1, C?.1, C?.1, U?.24 (VDD1), U?.36 (VDDIO2), U?.48 (VDD2), U?.9 (VDDA)
- new net GND: C?.2, C?.2, C?.2, C?.2, C?.2, C?.2, C?.2, C?.2, C?.2, C?.2, U?.23 (VSS1), U?.35 (VSS2), U?.47 (VSS3), U?.8 (VSSA)
Other:
- note added: "VDD1"
- note added: "VDD2"
- note added: "VDDA\n"
- note added: "VDDIO2\n"
